File: EAGLE/mspfacedraft3.sch (EAGLE design)
At the start: 26 parts, among them M1 G1040003D_LRA, P1 POT

Commit message: Schematic/brd updates/fixes
Parts:
- removed JP1, JP2, JP3, JP4, POTS6: (no value), SparkFun:M04LOCK
- removed M1: G1040003D_LRA, TEMP:G1040003D_LRA
- removed U$1: MSP430G2XX3TSSOP, ELEC327:MSP430G2XX3TSSOP
- removed U$6: SWITCH_DPDT, ELEC327:SWITCH_DPDT
- added BATT: M02, mspfacedraft3:M02
- added HAPTIC: G1040003D_LRA, TEMP:G1040003D_LRA
- added LEDOUT, PROGRAM: (no value), SparkFun:M04LOCK
- added MSP430: MSP430G2XX3TSSOP, ELEC327:MSP430G2XX3TSSOP
- added POTS: M06, mspfacedraft3:M06
- added SWITCH: SWITCH_DPDT, ELEC327:SWITCH_DPDT
Connections:
- removed net N$20: P1.S, U$1.2
- removed net N$7: LED1.DI, U$1.4
- removed net N$8: LED1.CI, U$1.6
- removed net P2.1: U$1.9
- new net CI: LED1.CI, MSP430.6
- new net DI: LED1.DI, MSP430.4
- new net POT1: MSP430.2, P1.S
- new net VBAT: C1.2, C2.2, LED10.EN, LED10.MODE, LED10.PVIN_1, LED10.PVIN_2, LED10.PVIN_3, LED10.PVIN_4, LED10.VIN, SWITCH.1, SWITCH.4
- net GND: now also BATT.1, HAPTIC.PIN2, LEDOUT.1, MSP430.20, POTS.1, PROGRAM.1; no longer JP1.1, JP2.1, JP3.1, JP4.1, M1.PIN2, POTS6.1, POTS6.2, U$1.20
- net OUT1: now also LEDOUT.4; no longer JP2.4
- net OUT2: now also LEDOUT.3; no longer JP2.3
- net P2.0: now also HAPTIC.PIN1, MSP430.8; no longer M1.PIN1, U$1.8
- net POT2: now also MSP430.3, POTS.6; no longer JP3.4, U$1.3
- net POT3: now also MSP430.5, POTS.5; no longer JP3.3, U$1.5
- net POT4: now also MSP430.7, POTS.4; no longer JP3.2, U$1.7
- net POT5: now also MSP430.14, POTS.3; no longer POTS6.3, U$1.14
- net POT6: now also MSP430.15, POTS.2; no longer POTS6.4, U$1.15
- net RST: now also MSP430.16, PROGRAM.3; no longer JP1.3, U$1.16
- net TEST: now also MSP430.17, PROGRAM.4; no longer JP1.4, U$1.17
- net VCC: now also LED10.VOUT_2, LED10.VOUT_3, LED10.VOUT_4, LEDOUT.2, MSP430.1, PROGRAM.2; no longer C1.2, C2.2, JP1.2, JP2.2, JP4.3, LED10.EN, LED10.MODE, LED10.PVIN_1, LED10.VIN, U$1.1, U$6.1, U$6.4
- net VINBAT: now also BATT.2, SWITCH.2, SWITCH.5; no longer JP4.4, U$6.2, U$6.5
Other:
- note added: "Bat Input + Switch"
- note added: "Haptics"
- note added: "Headers"
- note added: "LED Array"
- note added: "MSP430"
- note added: "Potentiometer"
- note added: "Voltage Regulator"
- moved on the sheet: C1, C2, C3, C4, CSUPPLY, L1, LED10, P1, R1
